Commit message: added end-effector tracking controller

File: kinova_description/urdf/d435_sensor.xacro (robot description, xacro)
@@ -31,8 +31,10 @@
       </inertial>
     </link>
-    <joint name="${namespace}_d435_camera_joint" type="fixed">
+    <joint name="${namespace}_d435_camera_joint" type="revolute">
       <xacro:insert_block name="origin" />
       <parent link="${parent_link}" />
       <child link="${namespace}_d435_camera_link" />
+      <axis xyz="0 0 1"/>
+      <limit lower="0" upper="0" effort="0" velocity="0"/>
     </joint>
     <gazebo reference="${namespace}_d435_camera_link">

File: kinova_description/urdf/j2s7s300.xacro (robot description, xacro)
@@ -115,4 +115,9 @@
     <xacro:property name="joint_end_effector_origin_xyz" value="0 0 -0.1600" />
     <xacro:property name="joint_end_effector_origin_rpy" value="${J_PI} 0 ${J_PI/2}" />
+	<xacro:property name="joint_obj" value="object" />
+	<xacro:property name="joint_obj_type" value="revolute" />
+	<xacro:property name="joint_obj_axis_xyz" value="0 0 1" />
+	<xacro:property name="joint_obj_origin_xyz" value="0 0 -0.1145" />
+    <xacro:property name="joint_obj_origin_rpy" value="${J_PI} 0 0" />
     <xacro:macro name="j2s7s300" params="base_parent prefix:=j2s7s300">
         <xacro:gazebo_config robot_namespace="${prefix}"/>
@@ -150,4 +155,26 @@
 	  </xacro:optical_flow_macro>
 -->
+		<link name="${prefix}_grasp_object">
+            <visual>
+                <geometry>
+                    <cylinder radius="0.01" length="0.02"/>
+                </geometry>
+            </visual>
+            <collision>
+                <geometry>
+                    <cylinder radius="0.001" length="0.002"/>
+                </geometry>
+            </collision>
+			<inertial>
+		    	<origin xyz="0 0 1" rpy="0 0 0"/>
+		  		<mass value="0.0001"/>
+		  		<inertia
+					ixx="0.0001" ixy="0.0" ixz="0.0"
+					iyy="0.0001" iyz="0.0"
+					izz="0.0001"/>
+			</inertial>
+         </link>
+	    <xacro:kinova_armjoint joint_name="${prefix}_joint_obj" type="${joint_obj_type}" parent="${prefix}_link_7" child="${prefix}_grasp_object" joint_axis_xyz="${joint_obj_axis_xyz}" joint_origin_xyz="${joint_obj_origin_xyz}" joint_origin_rpy="${joint_obj_origin_rpy}" joint_lower_limit="0" joint_upper_limit="0" joint_velocity_limit="0" joint_torque_limit="0" fixed="false"/>
+<!--
 	  <xacro:d435_macro
 		namespace="${prefix}"
@@ -162,4 +189,5 @@
 		<origin xyz="0.0 0.0 -0.04" rpy="0.0 ${-pi/2} ${pi}" />
 	  </xacro:d435_macro>
+-->
 		<gazebo>
 		 <plugin name="gazebo_grasp_fix" filename="libgazebo_grasp_fix.so">

Commit message: target approaching controller working v0

File: kinova_description/urdf/d435_sensor.xacro (robot description, xacro)
@@ -31,5 +31,5 @@
       </inertial>
     </link>
-    <joint name="${namespace}_d435_camera_joint" type="revolute">
+    <joint name="${namespace}_d435_camera_joint" type="fixed">
       <xacro:insert_block name="origin" />
       <parent link="${parent_link}" />

File: kinova_description/urdf/j2s7s300.xacro (robot description, xacro)
@@ -155,4 +155,5 @@
 	  </xacro:optical_flow_macro>
 -->
+<!--
 		<link name="${prefix}_grasp_object">
             <visual>
@@ -176,5 +177,5 @@
          </link>
 	    <xacro:kinova_armjoint joint_name="${prefix}_joint_obj" type="${joint_obj_type}" parent="${prefix}_link_7" child="${prefix}_grasp_object" joint_axis_xyz="${joint_obj_axis_xyz}" joint_origin_xyz="${joint_obj_origin_xyz}" joint_origin_rpy="${joint_obj_origin_rpy}" joint_lower_limit="0" joint_upper_limit="0" joint_velocity_limit="0" joint_torque_limit="0" fixed="false"/>
-<!--
+-->
 	  <xacro:d435_macro
 		namespace="${prefix}"
@@ -189,5 +190,4 @@
 		<origin xyz="0.0 0.0 -0.04" rpy="0.0 ${-pi/2} ${pi}" />
 	  </xacro:d435_macro>
--->
 		<gazebo>
 		 <plugin name="gazebo_grasp_fix" filename="libgazebo_grasp_fix.so">
