Commit message: ecc upd of grasp-devel for rl

File: kinova_description/urdf/j2s7s300.xacro (robot description, xacro)
@@ -16,4 +16,5 @@
     <xacro:include filename="$(find kinova_description)/urdf/kinova_common.xacro" />
     <xacro:include filename="$(find kinova_description)/urdf/kinova_finger_set.xacro" />
+    <xacro:include filename="$(find kinova_description)/urdf/optical_flow_sensor.xacro" />
     <!-- Import all Gazebo-customization elements -->
     <xacro:include filename="$(find kinova_description)/urdf/kinova.gazebo" />
@@ -134,4 +135,40 @@
         <xacro:kinova_virtual_joint joint_name="${prefix}_joint_end_effector" type="${joint_end_effector_type}" parent="${prefix}_link_7" child="${prefix}_end_effector" joint_axis_xyz="${joint_end_effector_axis_xyz}" joint_origin_xyz="${joint_end_effector_origin_xyz}" joint_origin_rpy="${joint_end_effector_origin_rpy}" joint_lower_limit="0" joint_upper_limit="0"/>
         <xacro:kinova_3fingers link_hand="${prefix}_link_7" prefix="${prefix}_"/>
+	  <xacro:optical_flow_macro
+		namespace="${prefix}"
+		parent_link="${prefix}_end_effector"
+		frame_rate="30"
+		horizontal_fov="1.5"
+		image_width="640"
+		image_height="480"
+		enable_visual="1"
+		enable_mesh="1">
+		<cylinder radius="0.01" length="0.01"/>
+		<origin xyz="0.02 0.02 -0.065" rpy="0.0 ${-pi/2} 0.0" />
+	  </xacro:optical_flow_macro>
+		<gazebo>
+		 <plugin name="gazebo_grasp_fix" filename="libgazebo_grasp_fix.so">
+		    <arm>
+		       <arm_name>j2s7s300_arm</arm_name>
+		       <palm_link>${prefix}::${prefix}_link_7</palm_link>
+		       <gripper_link>${prefix}::${prefix}_link_finger_1</gripper_link>
+		       <gripper_link>${prefix}::${prefix}_link_finger_2</gripper_link>
+		       <gripper_link>${prefix}::${prefix}_link_finger_3</gripper_link>
+		       <gripper_link>${prefix}::${prefix}_link_finger_tip_1</gripper_link>
+		       <gripper_link>${prefix}::${prefix}_link_finger_tip_2</gripper_link>
+		       <gripper_link>${prefix}::${prefix}_link_finger_tip_3</gripper_link>
+		    </arm>
+		   <forces_angle_tolerance>100</forces_angle_tolerance>
+		   <update_rate>4</update_rate>
+		   <grip_count_threshold>1</grip_count_threshold>
+		   <max_grip_count>8</max_grip_count>
+		   <release_tolerance>0.005</release_tolerance>
+		   <disable_collisions_on_attach>false</disable_collisions_on_attach>
+		   <contact_topic>__default_topic__</contact_topic>
+		 </plugin>
+		</gazebo>
     </xacro:macro>
+	<gazebo>
+		<plugin name="gripper_ctrl" filename="libkinova_gripper_plugin.so"/>
+	</gazebo>
 </root>

File: kinova_description/urdf/kinova_common.xacro (robot description, xacro)
@@ -85,5 +85,5 @@
         </xacro:if>
         <origin xyz="${joint_origin_xyz}" rpy="${joint_origin_rpy}"/>
-        <dynamics damping="0.0" friction="0.0"/>
+        <dynamics damping="0.05" friction="0.0"/>
      </joint>
    <xacro:unless value="${fixed}">
@@ -101,11 +101,4 @@
      <gazebo reference="${joint_name}">
         <provideFeedback>true</provideFeedback>
-      </gazebo>
-      <gazebo>
-        <plugin name="ft_sensor" filename="libgazebo_ros_ft_sensor.so">
-          <updateRate>30.0</updateRate>
-          <topicName>${joint_name}_ft_sensor_topic</topicName>
-          <jointName>${joint_name}</jointName>
-        </plugin>
       </gazebo>
      </xacro:unless>

Commit message: ball detection msgs and proper vision handler

File: kinova_description/urdf/j2s7s300.xacro (robot description, xacro)
@@ -145,5 +145,5 @@
 		enable_mesh="1">
 		<cylinder radius="0.01" length="0.01"/>
-		<origin xyz="0.02 0.02 -0.065" rpy="0.0 ${-pi/2} 0.0" />
+		<origin xyz="0.0 0.02 -0.02" rpy="0.0 ${-pi/2} 0.0" />
 	  </xacro:optical_flow_macro>
 		<gazebo>

File: kinova_description/urdf/j2s7s300_platform.xacro (robot description, xacro)
@@ -19,5 +19,4 @@
       <collision>
         <origin xyz="0 0 0.14" rpy="0 0 0"/>
-        <origin xyz="0 0 0" rpy="0 0 1.57079632679"/>
         <geometry>
 		  <box size="0.8 0.9 0.28"/>
@@ -25,7 +24,10 @@
       </collision>
       <visual>
-        <origin xyz="0 0 0" rpy="0 0 1.57079632679"/>
+        <origin xyz="0 0 0.14" rpy="0 0 0"/>
         <geometry>
+		  <box size="0.8 0.9 0.28"/>
+<!--
           <mesh  filename="model://ridgeback/meshes/ridgeback.stl" scale="1 1 1"/>
+-->
         </geometry>
       </visual>
@@ -38,5 +40,5 @@
     <child link="root" />
     <parent link="base_link" />
-    <origin xyz="0 0 0.35" rpy="0 0 0" />
+    <origin xyz="0 0 0.29" rpy="0 0 0" />
   </joint>
   <xacro:property name="robot_root" value="root" />

File: kinova_description/urdf/optical_flow_sensor.xacro (robot description, xacro)
@@ -38,4 +38,5 @@
     <gazebo reference="${namespace}_flow_camera_link">
       <sensor type="camera" name="${namespace}_camera_flow">
+     	<visualize>true</visualize>
         <always_on>true</always_on>
         <update_rate>${frame_rate}</update_rate>
@@ -52,10 +53,10 @@
           </image>
           <clip>
-            <near>0.05</near>
+            <near>0.01</near>
             <far>10</far>
           </clip>
         </camera>
         <plugin name="${namespace}_camera_flow_controller" filename="libgazebo_ros_camera.so">
-					<alwaysOn>true</alwaysOn>
+			 <alwaysOn>true</alwaysOn>
 		      <updateRate>100.0</updateRate>
 		      <cameraName>camera_flow</cameraName>
@@ -94,5 +95,5 @@
     </link>
     <joint name="${namespace}_z_ranger_joint" type="revolute">
-      <origin xyz="0 0 -0.06" rpy="0 ${-pi/2} 0"/>
+      <origin xyz="0 -0.008 -0.04" rpy="0 ${-pi/2} 0"/>
       <parent link="${parent_link}" />
       <child link="${namespace}_z_ranger_link" />

Commit message: kinova w d435

File: kinova_description/urdf/j2s7s300.xacro (robot description, xacro)
@@ -17,4 +17,5 @@
     <xacro:include filename="$(find kinova_description)/urdf/kinova_finger_set.xacro" />
     <xacro:include filename="$(find kinova_description)/urdf/optical_flow_sensor.xacro" />
+    <xacro:include filename="$(find kinova_description)/urdf/d435_sensor.xacro" />
     <!-- Import all Gazebo-customization elements -->
     <xacro:include filename="$(find kinova_description)/urdf/kinova.gazebo" />
@@ -135,4 +136,5 @@
         <xacro:kinova_virtual_joint joint_name="${prefix}_joint_end_effector" type="${joint_end_effector_type}" parent="${prefix}_link_7" child="${prefix}_end_effector" joint_axis_xyz="${joint_end_effector_axis_xyz}" joint_origin_xyz="${joint_end_effector_origin_xyz}" joint_origin_rpy="${joint_end_effector_origin_rpy}" joint_lower_limit="0" joint_upper_limit="0"/>
         <xacro:kinova_3fingers link_hand="${prefix}_link_7" prefix="${prefix}_"/>
+<!--
 	  <xacro:optical_flow_macro
 		namespace="${prefix}"
@@ -147,4 +149,17 @@
 		<origin xyz="0.0 0.02 -0.02" rpy="0.0 ${-pi/2} 0.0" />
 	  </xacro:optical_flow_macro>
+-->
+	  <xacro:d435_macro
+		namespace="${prefix}"
+		parent_link="${prefix}_end_effector"
+		frame_rate="30"
+		horizontal_fov="1.5"
+		image_width="640"
+		image_height="480"
+		enable_visual="1"
+		enable_mesh="1">
+		<cylinder radius="0.01" length="0.01"/>
+		<origin xyz="0.0 0.0 -0.04" rpy="0.0 ${-pi/2} ${pi}" />
+	  </xacro:d435_macro>
 		<gazebo>
 		 <plugin name="gazebo_grasp_fix" filename="libgazebo_grasp_fix.so">

File: kinova_description/urdf/optical_flow_sensor.xacro (robot description, xacro)
@@ -38,5 +38,5 @@
     <gazebo reference="${namespace}_flow_camera_link">
       <sensor type="camera" name="${namespace}_camera_flow">
-     	<visualize>true</visualize>
+     	<visualize>false</visualize>
         <always_on>true</always_on>
         <update_rate>${frame_rate}</update_rate>
@@ -105,5 +105,5 @@
 		   <sensor type="ray" name="rangefinder">
 			  <pose>0 0 0 0 0 0</pose>
-			  <visualize>true</visualize>
+			  <visualize>false</visualize>
 			  <update_rate>30</update_rate>
 				<ray>
@@ -128,5 +128,5 @@
 	      </ray>
 	      <plugin name="gazebo_ros_head_hokuyo_controller" filename="libgazebo_ros_range.so">
-						<topicName>zranger</topicName>
+			<topicName>zranger</topicName>
             <frameName>${namespace}_z_ranger_link</frameName>
             <gaussianNoise>0.000</gaussianNoise>

Commit message: major flow-cam frame fixes

File: kinova_description/urdf/j2s7s300.xacro (robot description, xacro)
@@ -141,5 +141,4 @@
         <xacro:kinova_virtual_joint joint_name="${prefix}_joint_end_effector" type="${joint_end_effector_type}" parent="${prefix}_link_7" child="${prefix}_end_effector" joint_axis_xyz="${joint_end_effector_axis_xyz}" joint_origin_xyz="${joint_end_effector_origin_xyz}" joint_origin_rpy="${joint_end_effector_origin_rpy}" joint_lower_limit="0" joint_upper_limit="0"/>
         <xacro:kinova_3fingers link_hand="${prefix}_link_7" prefix="${prefix}_"/>
-<!--
 	  <xacro:optical_flow_macro
 		namespace="${prefix}"
@@ -152,7 +151,6 @@
 		enable_mesh="1">
 		<cylinder radius="0.01" length="0.01"/>
-		<origin xyz="0.0 0.02 -0.02" rpy="0.0 ${-pi/2} 0.0" />
+		<origin xyz="0.0 0.02 -0.024" rpy="0.0 ${-pi/2} ${-pi}" />
 	  </xacro:optical_flow_macro>
--->
 <!--
 		<link name="${prefix}_grasp_object">
@@ -178,4 +176,5 @@
 	    <xacro:kinova_armjoint joint_name="${prefix}_joint_obj" type="${joint_obj_type}" parent="${prefix}_link_7" child="${prefix}_grasp_object" joint_axis_xyz="${joint_obj_axis_xyz}" joint_origin_xyz="${joint_obj_origin_xyz}" joint_origin_rpy="${joint_obj_origin_rpy}" joint_lower_limit="0" joint_upper_limit="0" joint_velocity_limit="0" joint_torque_limit="0" fixed="false"/>
 -->
+<!--
 	  <xacro:d435_macro
 		namespace="${prefix}"
@@ -190,4 +189,5 @@
 		<origin xyz="0.0 0.0 -0.04" rpy="0.0 ${-pi/2} ${pi}" />
 	  </xacro:d435_macro>
+-->
 		<gazebo>
 		 <plugin name="gazebo_grasp_fix" filename="libgazebo_grasp_fix.so">

File: kinova_description/urdf/optical_flow_sensor.xacro (robot description, xacro)
@@ -7,5 +7,5 @@
     <link name="${namespace}_flow_camera_link">
       <collision>
-        <origin xyz="0 0 0" rpy="0 0 0" />
+        <origin xyz="-0.015 0 0" rpy="0 0 0" />
         <geometry>
           <xacro:insert_block name="geometry" />
@@ -14,5 +14,5 @@
       <xacro:if value="${enable_visual}">
         <visual>
-          <origin xyz="0 0 0" rpy="0 0 ${-pi/2}" />
+          <origin xyz="0 0.02 0" rpy="0 0 ${-pi/2}" />
           <geometry>
           	<xacro:if value="${enable_mesh}">
@@ -35,4 +35,10 @@
       <parent link="${parent_link}" />
       <child link="${namespace}_flow_camera_link" />
+    </joint>
+    <link name="${namespace}_flow_camera_optical_link"/>
+    <joint name="${namespace}_flow_camera_optical_joint" type="fixed">
+      <origin xyz="0 0 0" rpy="${pi/2} ${pi} ${pi/2}"/>
+      <parent link="${namespace}_flow_camera_link"/>
+      <child link="${namespace}_flow_camera_optical_link"/>
     </joint>
     <gazebo reference="${namespace}_flow_camera_link">
@@ -63,5 +69,5 @@
 		      <imageTopicName>image_raw</imageTopicName>
 		      <cameraInfoTopicName>camera_info</cameraInfoTopicName>
-		      <frameName>${namespace}_flow_camera_link</frameName>
+		      <frameName>${namespace}_flow_camera_optical_link</frameName>
 		      <hackBaseline>0.07</hackBaseline>
 		      <distortionK1>0.0</distortionK1>
@@ -95,5 +101,5 @@
     </link>
     <joint name="${namespace}_z_ranger_joint" type="revolute">
-      <origin xyz="0 -0.008 -0.04" rpy="0 ${-pi/2} 0"/>
+      <origin xyz="0 0.012 -0.04" rpy="0 ${-pi/2} 0"/>
       <parent link="${parent_link}" />
       <child link="${namespace}_z_ranger_link" />
@@ -105,5 +111,5 @@
 		   <sensor type="ray" name="rangefinder">
 			  <pose>0 0 0 0 0 0</pose>
-			  <visualize>false</visualize>
+			  <visualize>true</visualize>
 			  <update_rate>30</update_rate>
 				<ray>
